File: grounding_device.kicad_sch (KiCad schematic)
At the start: 140 parts, among them IC1 NE555P, IC2 NE555P, IC3 NE555P, IC4 NE555P, Q1 2N2222, Q10 2N2222, Q11 2N2222, Q12 2N2222, Q2 2N2222, Q3 2N2222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

Commit message: Upgrade
Parts:
- added C28: 1uF, symbol PCM_Elektuur:C
- added R60: 2Om, symbol PCM_Elektuur:R
Connections:
- net 0: now also R60.1 (+)
- net Filters/Ground: now also C28.1 (+)
- new net: C28.2 (-), R60.2 (-)
Changed lines of the file:
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@@
 	)
 	(junction
+		(at 134.62 135.89)
+		(diameter 0)
+		(color 0 0 0 0)
+	)
+	(junction
 		(at 77.47 52.07)
 		(diameter 0)
@@
 	)
 	(junction
+		(at 156.21 167.64)
+		(diameter 0)
+		(color 0 0 0 0)
+	)
+	(junction
 		(at 170.18 176.53)
 		(diameter 0)
@@
 	(wire
 		(pts
+			(xy 134.62 135.89) (xy 134.62 153.67)
+		)
+		(stroke
+			(width 0)
+			(type default)
+		)
+	)
+	(wire
+		(pts
 			(xy 264.16 63.5) (xy 264.16 66.04)
 		)
@@
 	(wire
 		(pts
-			(xy 156.21 167.64) (xy 165.1 167.64)
-		)
-		(stroke
-			(width 0)
-			(type default)
-		)
-	)
-	(wire
-		(pts
 			(xy 224.79 69.85) (xy 208.28 69.85)
 		)
@@
 	(wire
 		(pts
-			(xy 134.62 130.81) (xy 134.62 153.67)
+			(xy 134.62 130.81) (xy 134.62 135.89)
 		)
 		(stroke
@@
 	(wire
 		(pts
+			(xy 142.24 167.64) (xy 156.21 167.64)
+		)
+		(stroke
+			(width 0)
+			(type default)
+		)
+	)
+	(wire
+		(pts
 			(xy 90.17 92.71) (xy 162.56 92.71)
 		)
@@
 	(wire
 		(pts
+			(xy 156.21 167.64) (xy 165.1 167.64)
+		)
+		(stroke
+			(width 0)
+			(type default)
+		)
+	)
+	(wire
+		(pts
 			(xy 229.87 29.21) (xy 229.87 30.48)
 		)
@@
 	(wire
 		(pts
+			(xy 142.24 135.89) (xy 134.62 135.89)
+		)
+		(stroke
+			(width 0)
+			(type default)
+		)
+	)
+	(wire
+		(pts
 			(xy 151.13 62.23) (xy 151.13 83.82)
 		)
@@
 	(wire
 		(pts
+			(xy 142.24 160.02) (xy 142.24 167.64)
+		)
+		(stroke
+			(width 0)
+			(type default)
+		)
+	)
+	(wire
+		(pts
 			(xy 246.38 127) (xy 261.62 127)
 		)
@@
 	(wire
 		(pts
+			(xy 142.24 139.7) (xy 142.24 135.89)
+		)
+		(stroke
+			(width 0)
+			(type default)
+		)
+	)
+	(wire
+		(pts
 			(xy 33.02 182.88) (xy 45.72 182.88)
 		)
@@
 	)
 	(symbol
+		(lib_id "PCM_Elektuur:R")
+		(at 142.24 154.94 180)
+		(unit 1)
+		(exclude_from_sim no)
+		(in_bom yes)
+		(on_board yes)
+		(dnp no)
+		(fields_autoplaced yes)
+		(property "Reference" "R60"
+			(at 144.78 153.6699 0)
+			(effects
+				(font
+					(size 1.27 1.27)
+				)
+				(justify right)
+			)
+		)
+		(property "Value" "2Om"
+			(at 144.78 156.2099 0)
+			(effects
+				(font
+					(size 1.27 1.27)
+				)
+				(justify right)
+			)
+		)
+		(property "Footprint" ""
+			(at 142.24 154.94 0)
+			(effects
+				(font
+					(size 1.27 1.27)
+				)
+				(hide yes)
+			)
+		)
+		(property "Datasheet" ""
+			(at 142.24 154.94 0)
+			(effects
+				(font
+					(size 1.27 1.27)
+				)
+				(hide yes)
+			)
+		)
+		(property "Description" ""
+			(at 142.24 154.94 0)
+			(effects
+				(font
+					(size 1.27 1.27)
+				)
+				(hide yes)
+			)
+		)
+		(property "Indicator" "+"
+			(at 145.415 158.115 0)
+			(effects
+				(font
+					(size 1.27 1.27)
+				)
+				(hide yes)
+			)
+		)
+		(property "Rating" "W"
+			(at 139.7 151.765 0)
+			(effects
+				(font
+					(size 1.27 1.27)
+				)
+				(justify left)
+				(hide yes)
+			)
+		)
+		(pin "1"
+		)
+		(pin "2"
+		)
+		(instances
+			(project "grounding_device"
+				(path "/63bcada5-65b5-4df8-beff-81b8339c1d00"
+					(reference "R60")
+					(unit 1)
+				)
+			)
+		)
+	)
+	(symbol
 		(lib_id "PCM_Elektuur:C")
 		(at 228.6 148.59 0)
@@
 					(unit 1)
 				)
+			)
+		)
+	)
+	(symbol
+		(lib_id "PCM_Elektuur:C")
+		(at 142.24 144.78 0)
+		(unit 1)
+		(exclude_from_sim no)
+		(in_bom yes)
+		(on_board yes)
+		(dnp no)
+		(fields_autoplaced yes)
+		(property "Reference" "C28"
+			(at 146.05 143.5099 0)
+			(effects
+				(font
+					(size 1.27 1.27)
+				)
+				(justify left)
+			)
+		)
+		(property "Value" "1uF"
+			(at 146.05 146.0499 0)
+			(effects
+				(font
+					(size 1.27 1.27)
+				)
+				(justify left)
+			)
+		)
+		(property "Footprint" ""
+			(at 142.24 144.78 0)
+			(effects
+				(font
+					(size 1.27 1.27)
+				)
+				(hide yes)
+			)
+		)
+		(property "Datasheet" ""
+			(at 142.24 144.78 0)
+			(effects
+				(font
+					(size 1.27 1.27)
+				)
+				(hide yes)
+			)
+		)
+		(property "Description" ""
+			(at 142.24 144.78 0)
+			(effects
+				(font
+					(size 1.27 1.27)
+				)
+				(hide yes)
+			)
+		)
+		(property "Indicator" "+"
+			(at 140.97 141.605 0)
+			(effects
+				(font
+					(size 1.27 1.27)
+				)
+				(hide yes)
+			)
+		)
+		(property "Rating" "V"
+			(at 141.605 147.955 0)
+			(effects
+				(font
+					(size 1.27 1.27)
+				)
+				(justify right)
+				(hide yes)
+			)
+		)
+		(pin "1"
+		)
+		(pin "2"
+		)
+		(instances
+			(project "grounding_device"
+				(path "/63bcada5-65b5-4df8-beff-81b8339c1d00"
+					(reference "C28")
+					(unit 1)
+				)

Commit message: Upgrade
Parts:
- added C29, C30: 220 pF, symbol PCM_Elektuur:C
- added R63: 1 Om, symbol PCM_Elektuur:R
Connections:
- net 0: now also C30.2 (-)
- net To Reley 5v line : now also C29.1 (+)
- net at C26.2 (-), C27.1 (+), R51.2 (-): now also R63.1 (+)
- new net: C29.2 (-), C30.1 (+), R63.2 (-)
Other:
- note added: "This filters must be soldering after resistors array to lines before place rele"
- note removed: "This 2 filters must be soldering after resistors array to (+)line before place rele"

Commit message: Upgrade
Parts:
- removed C28: 1uF, symbol PCM_Elektuur:C
- removed R19, R20, R21, R22, R32, R33, R34, R35, R42, R43, R44, R45, R46, R47, R48, R49: 680 Om - 5 kOM, symbol PCM_Elektuur:R
- removed R41: 10-9.5 MOM, symbol PCM_Elektuur:R
- added R64: 12-10-11-13kOm, symbol PCM_Elektuur:R
- added RV10, RV11, RV12, RV13, RV14, RV15, RV16, RV17, RV2, RV3, RV4, RV5, RV6, RV7, RV8, RV9: 10 kOm, symbol Device:R_Potentiometer_Small
- C13, C14, C20, C21: value 22 pF -> 9 pF
- C23, C25: value 100pF -> 100nF
- C26, C27: value 10pF -> 10nF
- R17, R50: value 1 Om -> 2 Om
- R39: value 10-9.5 MOM -> 2kOm
- R60: value 2Om -> 100kOm
Connections:
- net +5V: now also R60.1 (+), R64.1 (+), RV11.1, RV11.2, RV12.1, RV12.2, RV15.1, RV15.2, RV17.1, RV17.2, RV8.3
- net 0: now also R60.2 (-); no longer R60.1 (+)
- net 6 pin IC2: now also RV3.3
- net 6 pin IC3: now also RV4.3
- net 6 pin IC4: now also RV7.3
- net 8 pin IC2: now also RV2.1, RV2.2
- net 8 pin IC3: now also RV5.1, RV5.2
- net 8 pin IC4: now also RV6.1, RV6.2
- net At pin IC3: now also RV12.3, RV13.1, RV13.2
- net At pin IC4: now also RV10.1, RV10.2, RV11.3
- net Filters/Ground: now also R64.2 (-)
- net at S10.4: now also RV16.1, RV16.2, RV17.3
- net at S13.4: now also RV6.3, RV7.1, RV7.2
- net at S11.2: now also RV2.3, RV3.1, RV3.2
- net at C15.1, IC3.2 (TRIG), IC3.6 (THRES): now also RV13.3
- net at C1.1, IC2.2 (TRIG), IC2.6 (THRES): now also RV14.3
- net at C17.1, IC4.2 (TRIG), IC4.6 (THRES): now also RV10.3
- net at S12.4: now also RV4.1, RV4.2, RV5.3
- net at S11.4: now also RV14.1, RV14.2, RV15.3
- net at S10.2: now also RV8.1, RV8.2, RV9.3
- net at C3.1, IC1.2 (TRIG), IC1.6 (THRES): now also RV16.3, RV9.1, RV9.2
Other:
- moved on the sheet: R39

Commit message: Upgrade
Parts:
- added C28, C31: 820 pF, symbol PCM_Elektuur:C
- added C32, C33: ~820 nF, symbol PCM_Elektuur:C
- added R19, R20: 2 Om, symbol PCM_Elektuur:R
Connections:
- net 0: now also C31.2 (-), C33.2 (-)
- net Filters/Ground: now also R19.1 (+), R20.1 (+)
- net To Reley 5v line : now also C28.1 (+), C32.1 (+)
- new net: C32.2 (-), C33.1 (+), R20.2 (-)
- new net: C28.2 (-), C31.1 (+), R19.2 (-)
Other:
- moved on the sheet: C20, C21, C23, C25, R50, R62

Commit message: Upgarade
Parts:
- added C34, C35, C36, C37: 10uF, symbol PCM_Elektuur:C
- added L1, L2: L 10-15 coil turn, symbol Device:L_Ferrite_Coupled_Small_1324
Connections:
- net +5V: now also C36.1 (+), L1.1, L2.1
- net 0: now also C35.2 (-), C37.2 (-), L2.2
- new net: C35.1 (+), L1.4
- new net: C36.2 (-), L1.2, L2.3
- new net: C34.1 (+), L1.3
- new net: C34.2 (-), C37.1 (+), L2.4
Other:
- moved on the sheet: R1, R10, R11, R12, R13, R14, R15, R16, R2, R3, R4, R5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

Commit message: Upgrade
Parts:
- added R21, R22, R32, R33: ~100kOm, symbol Device:R_Small
Connections:
- net +5V: now also R21.1, R22.1, R32.1, R33.1
- net at IC1.3 (OUT), R25.1 (+), R55.1 (+)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: now also R21.2
- net at IC4.3 (OUT), R29.1 (+), R52.1 (+)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: now also R33.2
- net at IC3.3 (OUT), R24.1 (+), R53.1 (+)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: now also R32.2
- net at IC2.3 (OUT), R23.1 (+), R54.1 (+)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: now also R22.2

Commit message: Upgrade
Parts:
- removed R40: 10-9.5 MOM, symbol PCM_Elektuur:R
- added C38: 10 nF, symbol PCM_Elektuur:C
- added C39: 100 pF, symbol PCM_Elektuur:C
Connections:
- net +5V: now also C38.1 (+), C39.1 (+)
- net 0: now also C38.2 (-), C39.2 (-)
Changed lines of the file:
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@@
 	)
 	(junction
+		(at 264.16 48.26)
+		(diameter 0)
+		(color 0 0 0 0)
+	)
+	(junction
 		(at 127 162.56)
 		(diameter 0)
@@
 	)
 	(junction
+		(at 255.27 83.82)
+		(diameter 0)
+		(color 0 0 0 0)
+	)
+	(junction
 		(at 27.94 35.56)
 		(diameter 0)
@@
 	(wire
 		(pts
+			(xy 255.27 83.82) (xy 255.27 85.09)
+		)
+		(stroke
+			(width 0)
+			(type default)
+		)
+	)
+	(wire
+		(pts
 			(xy 213.36 24.13) (xy 213.36 21.59)
 		)
@@
 	(wire
 		(pts
+			(xy 276.86 74.93) (xy 276.86 85.09)
+		)
+		(stroke
+			(width 0)
+			(type default)
+		)
+	)
+	(wire
+		(pts
 			(xy 246.38 127) (xy 261.62 127)
 		)
@@
 	(wire
 		(pts
+			(xy 264.16 48.26) (xy 276.86 48.26)
+		)
+		(stroke
+			(width 0)
+			(type default)
+		)
+	)
+	(wire
+		(pts
 			(xy 226.06 107.95) (xy 226.06 120.65)
 		)
@@
 	(wire
 		(pts
+			(xy 276.86 48.26) (xy 276.86 64.77)
+		)
+		(stroke
+			(width 0)
+			(type default)
+		)
+	)
+	(wire
+		(pts
 			(xy 77.47 48.26) (xy 87.63 48.26)
 		)
@@
 	(wire
 		(pts
+			(xy 276.86 85.09) (xy 255.27 85.09)
+		)
+		(stroke
+			(width 0)
+			(type default)
+		)
+	)
+	(wire
+		(pts
 			(xy 68.58 66.04) (xy 83.82 66.04)
 		)
@@
 	(symbol
 		(lib_id "PCM_Elektuur:C")
+		(at 15.24 111.76 0)
+		(unit 1)
+		(exclude_from_sim no)
+		(in_bom yes)
+		(on_board yes)
+		(dnp no)
+		(fields_autoplaced yes)
+		(property "Reference" "C38"
+			(at 19.05 110.49 0)
+			(effects
+				(font
+					(size 1.27 1.27)
+				)
+				(justify left)
+			)
+		)
+		(property "Value" "10 nF"
+			(at 19.05 113.03 0)
+			(effects
+				(font
+					(size 1.27 1.27)
+				)
+				(justify left)
+			)
+		)
+		(property "Footprint" ""
+			(at 15.24 111.76 0)
+			(effects
+				(font
+					(size 1.27 1.27)
+				)
+				(hide yes)
+			)
+		)
+		(property "Datasheet" ""
+			(at 15.24 111.76 0)
+			(effects
+				(font
+					(size 1.27 1.27)
+				)
+				(hide yes)
+			)
+		)
+		(property "Description" ""
+			(at 15.24 111.76 0)
+			(effects
+				(font
+					(size 1.27 1.27)
+				)
+				(hide yes)
+			)
+		)
+		(property "Indicator" "+"
+			(at 13.97 108.585 0)
+			(effects
+				(font
+					(size 1.27 1.27)
+				)
+				(hide yes)
+			)
+		)
+		(property "Rating" "V"
+			(at 14.605 114.935 0)
+			(effects
+				(font
+					(size 1.27 1.27)
+				)
+				(justify right)
+				(hide yes)
+			)
+		)
+		(pin "1"
+		)
+		(pin "2"
+		)
+		(instances
+			(project "grounding_device"
+				(path "/63bcada5-65b5-4df8-beff-81b8339c1d00"
+					(reference "C38")
+					(unit 1)
+				)
+			)
+		)
+	)
+	(symbol
+		(lib_id "PCM_Elektuur:C")
 		(at 185.42 138.43 0)
 		(unit 1)
@@
 	)
 	(symbol
+		(lib_id "PCM_Elektuur:C")
+		(at 276.86 69.85 0)
+		(unit 1)
+		(exclude_from_sim no)
+		(in_bom yes)
+		(on_board yes)
+		(dnp no)
+		(property "Reference" "C39"
+			(at 280.162 69.596 0)
+			(effects
+				(font
+					(size 1.27 1.27)
+				)
+				(justify left)
+			)
+		)
+		(property "Value" "100 pF"
+			(at 277.622 72.898 0)
+			(effects
+				(font
+					(size 1.27 1.27)
+				)
+				(justify left)
+			)
+		)
+		(property "Footprint" ""
+			(at 276.86 69.85 0)
+			(effects
+				(font
+					(size 1.27 1.27)
+				)
+				(hide yes)
+			)
+		)
+		(property "Datasheet" ""
+			(at 276.86 69.85 0)
+			(effects
+				(font
+					(size 1.27 1.27)
+				)
+				(hide yes)
+			)
+		)
+		(property "Description" ""
+			(at 276.86 69.85 0)
+			(effects
+				(font
+					(size 1.27 1.27)
+				)
+				(hide yes)
+			)
+		)
+		(property "Indicator" "+"
+			(at 275.59 66.675 0)
+			(effects
+				(font
+					(size 1.27 1.27)
+				)
+				(hide yes)
+			)
+		)
+		(property "Rating" "V"
+			(at 276.225 73.025 0)
+			(effects
+				(font
+					(size 1.27 1.27)
+				)
+				(justify right)
+				(hide yes)
+			)
+		)
+		(pin "1"
+		)
+		(pin "2"
+		)
+		(instances
+			(project "grounding_device"
+				(path "/63bcada5-65b5-4df8-beff-81b8339c1d00"
+					(reference "C39")
+					(unit 1)
+				)
+			)
+		)
+	)
+	(symbol
 		(lib_id "PCM_Transistor_BJT_AKL:2N2222")
 		(at 40.64 38.1 0)
@@
 					(unit 1)
 				)
-			)
-		)
-	)
-	(symbol
-		(lib_id "PCM_Elektuur:R")
-		(at 15.24 111.76 0)
-		(unit 1)
-		(exclude_from_sim no)
-		(in_bom yes)
-		(on_board yes)
-		(dnp no)
-		(fields_autoplaced yes)
-		(property "Reference" "R40"
-			(at 17.78 110.49 0)
-			(effects
-				(font
-					(size 1.27 1.27)
-				)
-				(justify left)
-			)
-		)
-		(property "Value" "10-9.5 MOM"
-			(at 17.78 113.03 0)
-			(effects
-				(font
-					(size 1.27 1.27)
-				)
-				(justify left)
-			)
-		)
-		(property "Footprint" ""
-			(at 15.24 111.76 0)
-			(effects
-				(font
-					(size 1.27 1.27)
-				)
-				(hide yes)
-			)
-		)
-		(property "Datasheet" ""
-			(at 15.24 111.76 0)
-			(effects
-				(font
-					(size 1.27 1.27)
-				)
-				(hide yes)
-			)
-		)
-		(property "Description" ""
-			(at 15.24 111.76 0)
-			(effects
-				(font
-					(size 1.27 1.27)
-				)
-				(hide yes)
-			)
-		)
-		(property "Indicator" "+"
-			(at 12.065 108.585 0)
-			(effects
-				(font
-					(size 1.27 1.27)
-				)
-				(hide yes)
-			)
-		)
-		(property "Rating" "W"
-			(at 17.78 114.935 0)
-			(effects
-				(font
-					(size 1.27 1.27)
-				)
-				(justify left)
-				(hide yes)
-			)
-		)
-		(pin "1"
-		)
-		(pin "2"
-		)
-		(instances
-			(project "grounding_device"
-				(path "/63bcada5-65b5-4df8-beff-81b8339c1d00"
-					(reference "R40")
-					(unit 1)
-				)

Commit message: Upgrade
Parts:
- removed L1, L2: L 10-15 coil turn, symbol Device:L_Ferrite_Coupled_Small_1324
- added C40: 220 pF, symbol PCM_Elektuur:C
- added C41: 10nF, symbol PCM_Elektuur:C
- added C42: ~820 nF, symbol PCM_Elektuur:C
- added L1: L, symbol Device:L
- C35: value 10uF -> 9 pF
- C36: value 10uF -> 820 pF
- C37: value 10uF -> 100nF
Connections:
- net +5V: now also L1.2; no longer C36.1 (+)
- net 0: now also C34.2 (-), C36.2 (-), C40.2 (-), C41.2 (-), C42.2 (-)
- net at C35.1 (+): now also C34.1 (+), C36.1 (+), C37.1 (+), C40.1 (+), C41.1 (+), C42.1 (+), L1.1
