File: grounding_device.kicad_sch (KiCad schematic)
At the start: 163 parts, among them IC1 NE555P, IC2 NE555P, IC3 NE555P, IC4 NE555P, Q1 2N2222, Q10 2N2222, Q11 2N2222, Q12 2N2222, Q2 2N2222, Q3 2N2222, Q4 2N2222, Q5 2N2222, Q6 2N2222, Q7 2N2222, Q8 2N2222, Q9 2N2222

Commit message: Upgrade
Parts:
- removed C35: 9 pF, symbol PCM_Elektuur:C
- removed L1: L, symbol Device:L
Connections:
- net 0 is gone; now on net +5V: C1.2, C10.2, C11.2, C12.2, C14.2 (-), C15.2, C16.2 (-), C17.2, C18.2 (-), C19.2, C2.2 (-), C21.2 (-), C24.1 (+), C25.2 (-), C27.2 (-), C3.2, C30.2 (-), C31.2 (-), C33.2 (-), C34.2 (-), C36.2 (-), C37.2 (-), C38.2 (-), C39.2 (-), C4.2 (-), C40.2 (-), C41.2 (-), C42.2 (-), C5.2, C6.2, C7.2, C8.2, C9.2, IC1.1 (GND), IC2.1 (GND), IC3.1 (GND), IC4.1 (GND), Q1.1 (E), Q10.1 (E), Q11.1 (E), Q12.1 (E), Q2.1 (E), Q3.1 (E), Q4.1 (E), Q5.1 (E), Q6.1 (E), Q7.1 (E), Q8.1 (E), Q9.1 (E), R39.2 (-), R60.2 (-)
- net +5V: now also C34.1 (+), C36.1 (+), C37.1 (+), C40.1 (+), C41.1 (+), C42.1 (+)
Other:
- moved on the sheet: C34, C36, C37, C40, C41, C42

Commit message: Upgrade
Parts:
- added C35, C43, C44, C45, C46, C47, C48, C49: 47uF_5x5.3_16V, 4ms_Capacitor:CP_Elec_5x5.3, symbol PCM_4ms_Capacitor:47uF_5x5.3_16V
- added R34: 1-5 Om, symbol Device:R_Small
Connections:
- net +5V: now also C35.1, C43.1, C44.1, C45.1, C45.2, C46.1, C47.1, C48.1, C49.1, C49.2
- net Filters/Ground: now also R34.1
- new net: C35.2, C43.2, C44.2, C46.2, C47.2, C48.2, R34.2
Other:
- note added: "2024.12.09"

Commit message: Upgrade
Parts:
- removed C38: 10 nF, symbol PCM_Elektuur:C
- removed C39: 100 pF, symbol PCM_Elektuur:C

Commit message: Upgrade
Other:
- note added: "if you will to connect hight loaded AC devcie use different ground for internal GD filters."
Changed lines of the file:
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@@
+		)
+	)
+	(text "if you will to connect hight loaded \nAC devcie use different ground \nfor internal GD filters."
+		(exclude_from_sim no)
+		(at 145.034 136.652 0)
+		(effects
+			(font
+				(size 1.27 1.27)
+			)
 		)
 	)

Commit message: Upgrade
Parts:
- added R35: 10kOm, symbol Device:R_Small
- added U2: VOS618A, Package_SO:SSOP-4_4.4x2.6mm_P1.27mm, symbol Isolator:VOS618A
Connections:
- net +5V: now also R35.2, U2.2; no longer D1.1 (K), D2.1 (K), D3.1 (K), D4.1 (K), D5.1 (K), D6.1 (K), D7.1 (K), D8.1 (K), Re1.1 (+), Re2.1 (+), Re3.1 (+), Re4.1 (+), Re5.1 (+), Re6.1 (+), Re7.1 (+), Re8.1 (+)
- net at R25.2 (-): now also U2.1; no longer Q2.2 (B)
- net at D3.2 (A), Q2.3 (C), Re1.2 (-): now also U2.4
- new net: Q2.2 (B), R35.1, U2.3
- new net +5V Must be separate fom logic: D1.1 (K), D2.1 (K), D3.1 (K), D4.1 (K), D5.1 (K), D6.1 (K), D7.1 (K), D8.1 (K), Re1.1 (+), Re2.1 (+), Re3.1 (+), Re4.1 (+), Re5.1 (+), Re6.1 (+), Re7.1 (+), Re8.1 (+)
Other:
- note added: "Optocoupler"
- note added: "To separate rele supply ground"
- note added: "to logic ground"
- moved on the sheet: R25

Commit message: Upgrade
Parts:
- removed C10, C12, C35, C43, C44, C45, C46, C47, C48, C49, C8, C9: 47uF_5x5.3_16V, 4ms_Capacitor:CP_Elec_5x5.3, symbol PCM_4ms_Capacitor:47uF_5x5.3_16V
- removed D1, D2, D4, D5: 1N4004, Diode_THT_AKL:D_DO-41_SOD81_P7.62mm_Horizontal, symbol PCM_Diode_AKL:1N4004
- removed Q3, Q4, Q5, Q6: 2N2222, Package_TO_SOT_THT_AKL:TO-18-3_EBC, symbol PCM_Transistor_BJT_AKL:2N2222
- removed R11: 1-20 Om, symbol PCM_Generic:R,IEC
- removed R12, R13, R14, R15, R16: 1-12 Om, symbol PCM_Generic:R,IEC
- removed R26, R27, R28, R30: 1-6 kOm, symbol PCM_Elektuur:R
- removed R34: 1-5 Om, symbol Device:R_Small
- removed R52, R53, R54, R55: 1 kOm, symbol PCM_Elektuur:R
- removed Re4, Re5, Re6, Re7: 5V, symbol PCM_Elektuur:Re
- removed S6, S7, S8: S-changeover, symbol PCM_Elektuur:S-changeover
Other:
- note added: "In case of BIG EMI interference"
- note removed: "Resistor array must be created for first"

Commit message: Upgrade
Parts:
- added R11, R12, R13, R14: ~50-100kOm, symbol Device:R_Small
- C1, C15, C17, C3: Display 1000uF/16-10V -> 10-33uF/10-50V
Connections:
- net +5V: now also R11.2, R12.2, R13.2, R14.2
- net at C18.1 (+), IC4.5 (CONT): now also R14.1
- net at C16.1 (+), IC3.5 (CONT): now also R13.1
- net at C2.1 (+), IC1.5 (CONT): now also R11.1
- net at C4.1 (+), IC2.5 (CONT): now also R12.1

Commit message: Upgrade
Parts:
- C1, C15, C17, C3: Display 10-33uF/10-50V -> 1-33uF/10-50V
Changed lines of the file:
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@@
 			)
 		)
-		(property "Display" "10-33uF/10-50V"
+		(property "Display" "1-33uF/10-50V"
 			(at 99.06 77.0382 0)
 			(effects
@@
 			)
 		)
-		(property "Display" "10-33uF/10-50V"
+		(property "Display" "1-33uF/10-50V"
 			(at 161.29 77.0382 0)
 			(effects
@@
 			)
 		)
-		(property "Display" "10-33uF/10-50V"
+		(property "Display" "1-33uF/10-50V"
 			(at 36.83 77.0382 0)
 			(effects
@@
 			)
 		)
-		(property "Display" "10-33uF/10-50V"
+		(property "Display" "1-33uF/10-50V"
 			(at 223.52 77.0382 0)
 			(effects
